File: DP_Driver.sch (KiCad schematic (older format))
At the start: 16 parts, among them U201 PCA9685PW

Commit message: Updated Documentation Rev 1.0.0
- Finished Critical Fabrication Dimensions.
- Added Comments about Board.
Parts:
- R201, R202, R203, R204, R205, R206, R208, R209, R210, R211, R212, R213: value 1K -> 1k
Changed lines of the file:
@@
 EESchema Schematic File Version 4
+LIBS:ClockRadio_6x18SegDisp_I2C-cache
 EELAYER 26 0
 EELAYER END
@@
 AR Path="/5CC77626/5CC77B4B" Ref="R213"  Part="1"
 F 0 "R213" H 5350 4450 50  0000 L CNN
-F 1 "1K" H 5350 4350 50  0000 L CNN
+F 1 "1k" H 5350 4350 50  0000 L CNN
 F 2 "Resistor_SMD:R_0603_1608Metric" H 5300 4400 50  0001 C CNN
 F 3 "~" H 5300 4400 50  0001 C CNN
@@
 AR Path="/5CC77626/5CC77B44" Ref="R211"  Part="1"
 F 0 "R211" H 5050 4450 50  0000 L CNN
-F 1 "1K" H 5050 4350 50  0000 L CNN
+F 1 "1k" H 5050 4350 50  0000 L CNN
 F 2 "Resistor_SMD:R_0603_1608Metric" H 5000 4400 50  0001 C CNN
 F 3 "~" H 5000 4400 50  0001 C CNN
@@
 AR Path="/5CC77626/5CC77B3D" Ref="R209"  Part="1"
 F 0 "R209" H 4750 4450 50  0000 L CNN
-F 1 "1K" H 4750 4350 50  0000 L CNN
+F 1 "1k" H 4750 4350 50  0000 L CNN
 F 2 "Resistor_SMD:R_0603_1608Metric" H 4700 4400 50  0001 C CNN
 F 3 "~" H 4700 4400 50  0001 C CNN
@@
 AR Path="/5CC77626/5CC77B36" Ref="R206"  Part="1"
 F 0 "R206" H 4450 4450 50  0000 L CNN
-F 1 "1K" H 4450 4350 50  0000 L CNN
+F 1 "1k" H 4450 4350 50  0000 L CNN
 F 2 "Resistor_SMD:R_0603_1608Metric" H 4400 4400 50  0001 C CNN
 F 3 "~" H 4400 4400 50  0001 C CNN
@@
 AR Path="/5CC77626/5CC77B2F" Ref="R204"  Part="1"
 F 0 "R204" H 4150 4450 50  0000 L CNN
-F 1 "1K" H 4150 4350 50  0000 L CNN
+F 1 "1k" H 4150 4350 50  0000 L CNN
 F 2 "Resistor_SMD:R_0603_1608Metric" H 4100 4400 50  0001 C CNN
 F 3 "~" H 4100 4400 50  0001 C CNN
@@
 AR Path="/5CC77626/5CC77B28" Ref="R202"  Part="1"
 F 0 "R202" H 3850 4450 50  0000 L CNN
-F 1 "1K" H 3850 4350 50  0000 L CNN
+F 1 "1k" H 3850 4350 50  0000 L CNN
 F 2 "Resistor_SMD:R_0603_1608Metric" H 3800 4400 50  0001 C CNN
 F 3 "~" H 3800 4400 50  0001 C CNN
@@
 AR Path="/5CC77626/5CC77B21" Ref="R201"  Part="1"
 F 0 "R201" H 3850 3450 50  0000 L CNN
-F 1 "1K" H 3850 3350 50  0000 L CNN
+F 1 "1k" H 3850 3350 50  0000 L CNN
 F 2 "Resistor_SMD:R_0603_1608Metric" H 3800 3400 50  0001 C CNN
 F 3 "~" H 3800 3400 50  0001 C CNN
@@
 AR Path="/5CC77626/5CC77B1A" Ref="R203"  Part="1"
 F 0 "R203" H 4150 3450 50  0000 L CNN
-F 1 "1K" H 4150 3350 50  0000 L CNN
+F 1 "1k" H 4150 3350 50  0000 L CNN
 F 2 "Resistor_SMD:R_0603_1608Metric" H 4100 3400 50  0001 C CNN
 F 3 "~" H 4100 3400 50  0001 C CNN
@@
 AR Path="/5CC77626/5CC77B13" Ref="R205"  Part="1"
 F 0 "R205" H 4450 3450 50  0000 L CNN
-F 1 "1K" H 4450 3350 50  0000 L CNN
+F 1 "1k" H 4450 3350 50  0000 L CNN
 F 2 "Resistor_SMD:R_0603_1608Metric" H 4400 3400 50  0001 C CNN
 F 3 "~" H 4400 3400 50  0001 C CNN
@@
 AR Path="/5CC77626/5CC77B0C" Ref="R208"  Part="1"
 F 0 "R208" H 4750 3450 50  0000 L CNN
-F 1 "1K" H 4750 3350 50  0000 L CNN
+F 1 "1k" H 4750 3350 50  0000 L CNN
 F 2 "Resistor_SMD:R_0603_1608Metric" H 4700 3400 50  0001 C CNN
 F 3 "~" H 4700 3400 50  0001 C CNN
@@
 AR Path="/5CC77626/5CC77B05" Ref="R210"  Part="1"
 F 0 "R210" H 5050 3450 50  0000 L CNN
-F 1 "1K" H 5050 3350 50  0000 L CNN
+F 1 "1k" H 5050 3350 50  0000 L CNN
 F 2 "Resistor_SMD:R_0603_1608Metric" H 5000 3400 50  0001 C CNN
 F 3 "~" H 5000 3400 50  0001 C CNN
@@
 AR Path="/5CC77626/5CC77A89" Ref="R212"  Part="1"
 F 0 "R212" H 5350 3450 50  0000 L CNN
-F 1 "1K" H 5350 3350 50  0000 L CNN
+F 1 "1k" H 5350 3350 50  0000 L CNN
 F 2 "Resistor_SMD:R_0603_1608Metric" H 5300 3400 50  0001 C CNN
 F 3 "~" H 5300 3400 50  0001 C CNN
