File: ClockRadio_6x18SegDisp_I2C.kicad_pcb (KiCad board)
At the start: 4 copper layers, 315.2 x 69.9 mm, 296 parts, among them J101 SYSTEM, J102 5A, J103 Voltage_Selection, Q101 FDS6681Z, U101 TPS562219A, U102 TSL2591, U201 PCA9685PW, U301 PCA9685PW, U302 BL-S230B, U401 PCA9685PW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

Commit message: Updated Documentation Rev 1.0.0
- Finished Critical Fabrication Dimensions.
- Added Comments about Board.
Parts:
- R201, R202, R203, R204, R205, R206, R208, R209, R210, R211, R212, R213: value 1K -> 1k
- R301, R401, R501, R601, R701, R801: value 1k -> 1K
Other:
- board text added: "Board Dimensions: 12 in x 2.75 in Hole Dimensions Center -> 0.28 in from edge. Seperation -> 11.85 in x 2.19 Display Dimensions: 1.875 in x 2.75 in"
- board text added: "Displays: (x6) 16+2DP Segment. Drivers: (x6, Segments) 16 Drive, 6V tolerant, I2C controlled. (x1, DP) 16 Drive, 6V tolerant, I2C controlled. Misc. (x1) Lux sensor, I2C controlled (x1) Power FET for reverse Voltage Protection"
- board text added: "Power: INPUT -> 6 VDC @ TBD A. Regulated -> 3.3 VDC @ TBD A."

Commit message: Post assembly updates. Added pullup, R1001, for LUX sensor INT line. Changed R104 to 1k resolving issue.
Parts:
- added R1001: 1k, Resistor_SMD:R_0603_1608Metric, B.Cu at (60.7, 84.6)
- J101: value SYSTEM -> Display_tether
- R104: value 10k -> 1k
- moved C105 1.31 mm to (347.1, 54.0), turned to 270 degrees
- moved C106 0.95 mm to (345.5, 54.0), turned to 270 degrees
- moved U102 0.25 mm to (346.3, 54.0), turned to 0 degrees
Connections:
- net Net-(R314-Pad2) renamed /Display_0/LED1
- net Net-(R315-Pad2) renamed /Display_0/LED3
- net Net-(R316-Pad2) renamed /Display_0/LED6
- net Net-(R317-Pad2) renamed /Display_0/LED4
- net Net-(R318-Pad2) renamed /Display_0/LED11
- net Net-(R319-Pad2) renamed /Display_0/LED9
- net Net-(R320-Pad2) renamed /Display_0/LED12
- net Net-(R321-Pad2) renamed /Display_0/LED14
- net Net-(R323-Pad2) renamed /Display_0/LED0
- net Net-(R324-Pad2) renamed /Display_0/LED2
- net Net-(R325-Pad2) renamed /Display_0/LED7
- net Net-(R326-Pad2) renamed /Display_0/LED5
- net Net-(R327-Pad2) renamed /Display_0/LED10
- net Net-(R328-Pad2) renamed /Display_0/LED8
- net Net-(R329-Pad2) renamed /Display_0/LED13
- net Net-(R330-Pad2) renamed /Display_0/LED15
- net Net-(R414-Pad2) renamed /Display_1/LED1
- net Net-(R415-Pad2) renamed /Display_1/LED3
- net Net-(R416-Pad2) renamed /Display_1/LED6
- net Net-(R417-Pad2) renamed /Display_1/LED4
- net Net-(R418-Pad2) renamed /Display_1/LED11
- net Net-(R419-Pad2) renamed /Display_1/LED9
- net Net-(R420-Pad2) renamed /Display_1/LED12
- net Net-(R421-Pad2) renamed /Display_1/LED14
- net Net-(R423-Pad2) renamed /Display_1/LED0
- net Net-(R424-Pad2) renamed /Display_1/LED2
- net Net-(R425-Pad2) renamed /Display_1/LED7
- net Net-(R426-Pad2) renamed /Display_1/LED5
- net Net-(R427-Pad2) renamed /Display_1/LED10
- net Net-(R428-Pad2) renamed /Display_1/LED8
- net Net-(R429-Pad2) renamed /Display_1/LED13
- net Net-(R430-Pad2) renamed /Display_1/LED15
- net Net-(R514-Pad2) renamed /Display_2/LED1
- net Net-(R515-Pad2) renamed /Display_2/LED3
- net Net-(R516-Pad2) renamed /Display_2/LED6
- net Net-(R517-Pad2) renamed /Display_2/LED4
- net Net-(R518-Pad2) renamed /Display_2/LED11
- net Net-(R519-Pad2) renamed /Display_2/LED9
- net Net-(R520-Pad2) renamed /Display_2/LED12
- net Net-(R521-Pad2) renamed /Display_2/LED14
- net Net-(R523-Pad2) renamed /Display_2/LED0
- net Net-(R524-Pad2) renamed /Display_2/LED2
- net Net-(R525-Pad2) renamed /Display_2/LED7
- net Net-(R526-Pad2) renamed /Display_2/LED5
- net Net-(R527-Pad2) renamed /Display_2/LED10
- net Net-(R528-Pad2) renamed /Display_2/LED8
- net Net-(R529-Pad2) renamed /Display_2/LED13
- net Net-(R530-Pad2) renamed /Display_2/LED15
- net Net-(R614-Pad2) renamed /Display_3/LED1
- net Net-(R615-Pad2) renamed /Display_3/LED3
- net Net-(R616-Pad2) renamed /Display_3/LED6
- net Net-(R617-Pad2) renamed /Display_3/LED4
- net Net-(R618-Pad2) renamed /Display_3/LED11
- net Net-(R619-Pad2) renamed /Display_3/LED9
- net Net-(R620-Pad2) renamed /Display_3/LED12
- net Net-(R621-Pad2) renamed /Display_3/LED14
- net Net-(R623-Pad2) renamed /Display_3/LED0
- net Net-(R624-Pad2) renamed /Display_3/LED2
- net Net-(R625-Pad2) renamed /Display_3/LED7
- net Net-(R626-Pad2) renamed /Display_3/LED5
- net Net-(R627-Pad2) renamed /Display_3/LED10
- net Net-(R628-Pad2) renamed /Display_3/LED8
- net Net-(R629-Pad2) renamed /Display_3/LED13
- net Net-(R630-Pad2) renamed /Display_3/LED15
- net Net-(R714-Pad2) renamed /Display_4/LED1
- net Net-(R715-Pad2) renamed /Display_4/LED3
- net Net-(R716-Pad2) renamed /Display_4/LED6
- net Net-(R717-Pad2) renamed /Display_4/LED4
- net Net-(R718-Pad2) renamed /Display_4/LED11
- net Net-(R719-Pad2) renamed /Display_4/LED9
- net Net-(R720-Pad2) renamed /Display_4/LED12
- net Net-(R721-Pad2) renamed /Display_4/LED14
- net Net-(R723-Pad2) renamed /Display_4/LED0
- net Net-(R724-Pad2) renamed /Display_4/LED2
- net Net-(R725-Pad2) renamed /Display_4/LED7
- net Net-(R726-Pad2) renamed /Display_4/LED5
- net Net-(R727-Pad2) renamed /Display_4/LED10
- net Net-(R728-Pad2) renamed /Display_4/LED8
- net Net-(R729-Pad2) renamed /Display_4/LED13
- net Net-(R730-Pad2) renamed /Display_4/LED15
- net Net-(R814-Pad2) renamed /Diplay_5/LED1
- net Net-(R815-Pad2) renamed /Diplay_5/LED3
- net Net-(R816-Pad2) renamed /Diplay_5/LED6
- net Net-(R817-Pad2) renamed /Diplay_5/LED4
- net Net-(R818-Pad2) renamed /Diplay_5/LED11
- net Net-(R819-Pad2) renamed /Diplay_5/LED9
- net Net-(R820-Pad2) renamed /Diplay_5/LED12
- net Net-(R821-Pad2) renamed /Diplay_5/LED14
- net Net-(R823-Pad2) renamed /Diplay_5/LED0
- net Net-(R824-Pad2) renamed /Diplay_5/LED2
- net Net-(R825-Pad2) renamed /Diplay_5/LED7
- net Net-(R826-Pad2) renamed /Diplay_5/LED5
- net Net-(R827-Pad2) renamed /Diplay_5/LED10
- net Net-(R828-Pad2) renamed /Diplay_5/LED8
- net Net-(R829-Pad2) renamed /Diplay_5/LED13
- net Net-(R830-Pad2) renamed /Diplay_5/LED15
Routing:
- net /I2C_SDA: track 348.8 -> 351.8 mm
- net V3P3: track 109.8 -> 111.5 mm, vias 64 -> 65
- net /I2C_INT: track 315.7 -> 314.8 mm, vias 2 -> 3
- net /I2C_SCL: track 340.5 -> 339.7 mm
- net /CLK_EXT_GLOBAL: track 356.7 -> 357.4 mm
Other:
- board text added: "Power: INPUT -> 6 VDC @ 2.25 A. Regulated -> 3.3 VDC @ 0.07 A."
- board text removed: "Power: INPUT -> 6 VDC @ TBD A. Regulated -> 3.3 VDC @ TBD A."
