File: ClockRadio_6x18SegDisp_I2C.sch (KiCad schematic (older format))
At the start: 64 parts, among them J101 SYSTEM, J102 5A, J103 Voltage_Selection, Q101 FDS6681Z, U101 TPS562219A, U102 TSL2591

Commit message: Post assembly updates. Added pullup, R1001, for LUX sensor INT line. Changed R104 to 1k resolving issue.
Parts:
- added R1001: 1k, Resistor_SMD:R_0603_1608Metric, symbol Device:R_Small_US
- J101: value SYSTEM -> Display_tether
- R104: value 10k -> 1k
Connections:
- net I2C_INT: now also R1001.2
- net V3P3: now also R1001.1
Other:
- note added: "Voltage Selection\n1 & 2 <Barrel Jack> 3 & 4\n5 & 6 <V6P0_SYSTEM> 3 & 4"
- note removed: "Voltage Selection\n2 <=> 1 V6P0_SCREW\n2 <=> 3 V6P0_JACK\n2 <=> 5 V6P0_SYSTEM"
- moved on the sheet: R102, R103
Changed lines of the file:
@@
 L Device:R_Small_US R103
 U 1 1 5DDB7D02
-P 2700 4900
-F 0 "R103" H 2768 4946 50  0000 L CNN
-F 1 "1k" H 2768 4855 50  0000 L CNN
-F 2 "Resistor_SMD:R_0603_1608Metric" H 2700 4900 50  0001 C CNN
-F 3 "" H 2700 4900 50  0001 C CNN
-	1    2700 4900
+P 2800 4900
+F 0 "R103" H 2868 4946 50  0000 L CNN
+F 1 "1k" H 2868 4855 50  0000 L CNN
+F 2 "Resistor_SMD:R_0603_1608Metric" H 2800 4900 50  0001 C CNN
+F 3 "" H 2800 4900 50  0001 C CNN
+	1    2800 4900
 	1    0    0    -1
 $EndComp
@@
 L Device:R_Small_US R102
 U 1 1 5DDF72AA
-P 2300 4900
-F 0 "R102" H 2368 4946 50  0000 L CNN
-F 1 "1k" H 2368 4855 50  0000 L CNN
-F 2 "Resistor_SMD:R_0603_1608Metric" H 2300 4900 50  0001 C CNN
-F 3 "" H 2300 4900 50  0001 C CNN
-	1    2300 4900
+P 2400 4900
+F 0 "R102" H 2468 4946 50  0000 L CNN
+F 1 "1k" H 2468 4855 50  0000 L CNN
+F 2 "Resistor_SMD:R_0603_1608Metric" H 2400 4900 50  0001 C CNN
+F 3 "" H 2400 4900 50  0001 C CNN
+	1    2400 4900
 	1    0    0    -1
 $EndComp
@@
 I2C_INT
 Wire Wire Line
-	2700 5200 2700 5000
-Wire Wire Line
-	2700 4800 2700 4700
-Wire Wire Line
-	2700 4700 2300 4700
-Wire Wire Line
-	2300 4700 2300 4800
-Wire Wire Line
-	2300 5000 2300 5300
-Wire Wire Line
-	2300 5300 3000 5300
-Connection ~ 2300 4700
-Wire Wire Line
-	2300 4700 2300 4600
-Text GLabel 1500 4700 2    50   Output ~ 0
+	2800 5200 2800 5000
+Wire Wire Line
+	2800 4800 2800 4700
+Wire Wire Line
+	2800 4700 2400 4700
+Wire Wire Line
+	2400 4700 2400 4800
+Wire Wire Line
+	2400 5000 2400 5300
+Wire Wire Line
+	2400 5300 3000 5300
+Connection ~ 2400 4700
+Text GLabel 1400 4700 2    50   Output ~ 0
 V6P0_SYSTEM
 Text Label 5400 5400 0    50   ~ 10
@@
 CLK_EXT_GLOBAL
 Wire Wire Line
-	2700 5200 3000 5200
+	2800 5200 3000 5200
 Text Notes 1700 1200 2    50   ~ 10
 | |SYSTEM| |\n \/  V_IN  \/
@@
 Text Notes 1800 6400 0    250  ~ 50
 Logos
-Text Notes 4700 10400 0    150  ~ 30
+Text Notes 4500 10200 0    150  ~ 30
 I2C Address List\nLED0    0x81\nLED1    0x82\nLED2    0x83\nLED3    0x84\nLED4    0x85\nLED5    0x86\nLED6    0x87\nLED_DP  0x88\nLUX     0x29
 Connection ~ 5900 5400
 Wire Bus Line
 	5900 5400 9800 5400
-Text Notes 5800 7200 0    150  ~ 30
-Voltage Selection\n2 <=> 1    V6P0_SCREW\n2 <=> 3    V6P0_JACK\n2 <=> 5    V6P0_SYSTEM
+Text Notes 5500 6800 0    150  ~ 30
+Voltage Selection\n1 & 2 <Barrel Jack> 3 & 4\n5 & 6 <V6P0_SYSTEM> 3 & 4
 $Comp
 L ERW_Power:V6P0 #PWR0106
@@
 P 3800 2000
 F 0 "R104" H 4000 2100 50  0000 C CNN
-F 1 "10k" H 4000 2000 50  0000 C CNN
+F 1 "1k" H 4000 2000 50  0000 C CNN
 F 2 "Resistor_SMD:R_0603_1608Metric" H 3800 2000 50  0001 C CNN
 F 3 "" H 3800 2000 50  0001 C CNN
@@
 P 1000 5100
 F 0 "J101" H 1106 5678 50  0000 C CNN
-F 1 "SYSTEM" H 1106 5587 50  0000 C CNN
+F 1 "Display_tether" H 1106 5587 50  0000 C CNN
 F 2 "ERW_Conn:ESHF-105-01-L-D" H 1000 5100 50  0001 C CNN
 F 3 "" H 1000 5100 50  0001 C CNN
@@
 L ERW_Power:V3P3 #PWR0103
 U 1 1 5D2FEF32
-P 2300 4600
-F 0 "#PWR0103" H 2300 4450 50  0001 C CNN
-F 1 "V3P3" H 2315 4773 50  0000 C CNN
-F 2 "" H 2200 4350 50  0001 C CNN
-F 3 "" H 2300 4450 50  0001 C CNN
-	1    2300 4600
+P 2800 4600
+F 0 "#PWR0103" H 2800 4450 50  0001 C CNN
+F 1 "V3P3" H 2815 4773 50  0000 C CNN
+F 2 "" H 2700 4350 50  0001 C CNN
+F 3 "" H 2800 4450 50  0001 C CNN
+	1    2800 4600
 	1    0    0    -1
 $EndComp
@@
 	1300 4700 1200 4700
 Wire Wire Line
-	1300 4700 1500 4700
+	1300 4700 1400 4700
 Connection ~ 1300 4700
 Entry Wire Line
@@
 	3000 5400 1200 5400
 Wire Wire Line
-	2300 5300 1200 5300
-Connection ~ 2300 5300
-Wire Wire Line
-	2700 5200 1200 5200
-Connection ~ 2700 5200
-Wire Wire Line
-	3000 5100 1200 5100
+	2400 5300 1200 5300
+Connection ~ 2400 5300
+Wire Wire Line
+	2800 5200 1200 5200
+Connection ~ 2800 5200
+Wire Wire Line
+	3000 5100 2000 5100
 Connection ~ 4200 1500
 Connection ~ 3800 1500
@@
 Wire Notes Line
 	5100 2800 5100 7300
+$Comp
+L Device:R_Small_US R1001
+U 1 1 5D2944F6
+P 2000 4900
+F 0 "R1001" H 2068 4946 50  0000 L CNN
+F 1 "1k" H 2068 4855 50  0000 L CNN
+F 2 "Resistor_SMD:R_0603_1608Metric" H 2000 4900 50  0001 C CNN
+F 3 "" H 2000 4900 50  0001 C CNN
+	1    2000 4900
+	1    0    0    -1
+$EndComp
+Wire Wire Line
+	2000 4800 2000 4700
+Wire Wire Line
+	2000 4700 2400 4700
+Wire Wire Line
+	2800 4700 2800 4600
+Connection ~ 2800 4700
+Wire Wire Line
+	2000 5000 2000 5100
+Connection ~ 2000 5100
+Wire Wire Line
+	2000 5100 1200 5100
 Wire Bus Line
 	5900 4300 5900 5400
