File: Display.sch (KiCad schematic (older format))
At the start: 36 parts, among them U301 PCA9685PW, U302 BL-S230B

Commit message: Updated Documentation Rev 1.0.0
- Finished Critical Fabrication Dimensions.
- Added Comments about Board.
Parts:
- R301: value 1k -> 1K
Changed lines of the file:
@@
 EESchema Schematic File Version 4
+LIBS:ClockRadio_6x18SegDisp_I2C-cache
 EELAYER 26 0
 EELAYER END
@@
 AR Path="/5CC95B4E/5CD41A0A" Ref="R801"  Part="1"
 F 0 "R801" H 1550 3450 50  0000 L CNN
-F 1 "1k" H 1550 3350 50  0000 L CNN
+F 1 "1K" H 1550 3350 50  0000 L CNN
 F 2 "Resistor_SMD:R_0603_1608Metric" H 1500 3400 50  0001 C CNN
 F 3 "~" H 1500 3400 50  0001 C CNN

Commit message: Post assembly updates. Added pullup, R1001, for LUX sensor INT line. Changed R104 to 1k resolving issue.
Connections:
- net LED4: now reaches R817.2, U301.10 (LED4)
- net LED5: now reaches R826.2, U301.11 (LED5)
- net LED6: now reaches R816.2, U301.12 (LED6)
- net LED7: now reaches R825.2, U301.13 (LED7)
- net LED8: now reaches R828.2, U301.15 (LED8)
- net LED9: now reaches R819.2, U301.16 (LED9)
- net LED10: now reaches R827.2, U301.17 (LED10)
- net LED11: now reaches R818.2, U301.18 (LED11)
- net LED12: now reaches R820.2, U301.19 (LED12)
- net LED13: now reaches R829.2, U301.20 (LED13)
- net LED14: now reaches R821.2, U301.21 (LED14)
- net LED15: now reaches R830.2, U301.22 (LED15)
- net LED0: now reaches R823.2, U301.6 (LED0)
- net LED1: now reaches R814.2, U301.7 (LED1)
- net LED2: now reaches R824.2, U301.8 (LED2)
- net LED3: now reaches R815.2, U301.9 (LED3)
Changed lines of the file:
@@
 Wire Wire Line
 	7200 4500 7200 5600
+Text Label 5100 1700 0    50   ~ 0
+LED0
+Text Label 5200 1900 0    50   ~ 0
+LED1
+Text Label 5300 2100 0    50   ~ 0
+LED2
+Text Label 5000 3000 0    50   ~ 0
+LED3
+Text Label 5000 3100 0    50   ~ 0
+LED4
+Text Label 5000 3200 0    50   ~ 0
+LED5
+Text Label 5000 3300 0    50   ~ 0
+LED6
+Text Label 5000 3400 0    50   ~ 0
+LED7
+Text Label 5000 3500 0    50   ~ 0
+LED8
+Text Label 5000 3600 0    50   ~ 0
+LED9
+Text Label 5000 3700 0    50   ~ 0
+LED10
+Text Label 5000 3800 0    50   ~ 0
+LED11
+Text Label 5000 3900 0    50   ~ 0
+LED12
+Text Label 5000 4000 0    50   ~ 0
+LED13
+Text Label 5200 5000 0    50   ~ 0
+LED14
+Text Label 5100 5200 0    50   ~ 0
+LED15
 $EndSCHEMATC
